Commit message: 200713

File: urdf/aruco/turtlebot3_aruco_0.urdf.xacro (robot description, xacro)
@@ -75,5 +75,5 @@
         <mesh filename="package://turtlebot3_description/meshes/wheels/right_tire.stl" scale="0.001 0.001 0.001"/>
       </geometry>
-      <material name="dark"/>
+      <material name="dark" />
     </visual>
     <collision>
@@ -164,4 +164,73 @@
     </inertial>
   </link>
+<gazebo reference="ball">
+     <material>Marker/White</material>
+     <turnGravityOff>false</turnGravityOff>
+ </gazebo>
+  <link name="ball">
+    <visual>
+      <origin xyz="0 0 0" rpy="0 0 0"/>
+      <geometry>
+             <box size="0.15 0.15 01e-5"/>
+      </geometry>
+         <material name="m_Blue">
+    <color rgba="0.0 0.0 0.0 1.0"/>
+    <lighting>1</lighting>
+  </material>
+    </visual>
+    <collision>
+      <origin xyz="0.015 0 -0.0065" rpy="0 0 0"/>
+      <geometry>
+        <cylinder length="0.0315" radius="0.055"/>
+      </geometry>
+    </collision>
+    <inertial>
+      <mass value="0.114" />
+      <origin xyz="0 0 0" />
+      <inertia ixx="0.001" ixy="0.0" ixz="0.0"
+               iyy="0.001" iyz="0.0"
+               izz="0.001" />
+    </inertial>
+  </link>
+  <joint name="base_scan_ball" type="fixed">
+    <parent link="base_scan"/>
+    <child link="ball"/>
+    <origin xyz="-0.14 0.0 -0.03" rpy="0 1.57 0"/>
+    <axis xyz="0 0 1"/>
+  </joint>
+<gazebo reference="aruco">
+     <material>Marker/Marker0</material>
+     <turnGravityOff>false</turnGravityOff>
+ </gazebo>
+  <link name="aruco">
+    <visual>
+      <origin xyz="0 0 0" rpy="0 0 0"/>
+      <geometry>
+             <box size="0.12 0.12 1e-5"/>
+      </geometry>
+         <material name="m_Blue">
+    <color rgba="0.0 0.0 0.0 1.0"/>
+  </material>
+    </visual>
+    <collision>
+      <origin xyz="0.015 0 -0.0065" rpy="0 0 0"/>
+      <geometry>
+        <cylinder length="0.0315" radius="0.055"/>
+      </geometry>
+    </collision>
+    <inertial>
+      <mass value="0.114" />
+      <origin xyz="0 0 0" />
+      <inertia ixx="0.001" ixy="0.0" ixz="0.0"
+               iyy="0.001" iyz="0.0"
+               izz="0.001" />
+    </inertial>
+  </link>
+  <joint name="aruco_scan_ball" type="fixed">
+    <parent link="ball"/>
+    <child link="aruco"/>
+    <origin xyz="-0.0 0.0 -0.001" rpy="0 0 0"/>
+    <axis xyz="0 0 1"/>
+  </joint>
   <joint name="camera_joint" type="fixed">
     <origin xyz="0.064 -0.065 0.094" rpy="0 0 0"/>

File: urdf/aruco/turtlebot3_aruco_1.urdf.xacro (robot description, xacro)
@@ -75,5 +75,5 @@
         <mesh filename="package://turtlebot3_description/meshes/wheels/right_tire.stl" scale="0.001 0.001 0.001"/>
       </geometry>
-      <material name="dark"/>
+      <material name="dark" />
     </visual>
     <collision>
@@ -164,4 +164,73 @@
     </inertial>
   </link>
+<gazebo reference="ball">
+     <material>Marker/White</material>
+     <turnGravityOff>false</turnGravityOff>
+ </gazebo>
+  <link name="ball">
+    <visual>
+      <origin xyz="0 0 0" rpy="0 0 0"/>
+      <geometry>
+             <box size="0.15 0.15 1e-5"/>
+      </geometry>
+         <material name="m_Blue">
+    <color rgba="0.0 0.0 0.0 1.0"/>
+    <lighting>1</lighting>
+  </material>
+    </visual>
+    <collision>
+      <origin xyz="0.015 0 -0.0065" rpy="0 0 0"/>
+      <geometry>
+        <cylinder length="0.0315" radius="0.055"/>
+      </geometry>
+    </collision>
+    <inertial>
+      <mass value="0.114" />
+      <origin xyz="0 0 0" />
+      <inertia ixx="0.001" ixy="0.0" ixz="0.0"
+               iyy="0.001" iyz="0.0"
+               izz="0.001" />
+    </inertial>
+  </link>
+  <joint name="base_scan_ball" type="fixed">
+    <parent link="base_scan"/>
+    <child link="ball"/>
+    <origin xyz="-0.14 0.0 -0.03" rpy="0 1.57 0"/>
+    <axis xyz="0 0 1"/>
+  </joint>
+<gazebo reference="aruco">
+     <material>Marker/Marker1</material>
+     <turnGravityOff>false</turnGravityOff>
+ </gazebo>
+  <link name="aruco">
+    <visual>
+      <origin xyz="0 0 0" rpy="0 0 0"/>
+      <geometry>
+             <box size="0.12 0.12 1e-5"/>
+      </geometry>
+         <material name="m_Blue">
+    <color rgba="0.0 0.0 0.0 1.0"/>
+  </material>
+    </visual>
+    <collision>
+      <origin xyz="0.015 0 -0.0065" rpy="0 0 0"/>
+      <geometry>
+        <cylinder length="0.0315" radius="0.055"/>
+      </geometry>
+    </collision>
+    <inertial>
+      <mass value="0.114" />
+      <origin xyz="0 0 0" />
+      <inertia ixx="0.001" ixy="0.0" ixz="0.0"
+               iyy="0.001" iyz="0.0"
+               izz="0.001" />
+    </inertial>
+  </link>
+  <joint name="aruco_scan_ball" type="fixed">
+    <parent link="ball"/>
+    <child link="aruco"/>
+    <origin xyz="-0.0 0.0 -0.001" rpy="0 0 0"/>
+    <axis xyz="0 0 1"/>
+  </joint>
   <joint name="camera_joint" type="fixed">
     <origin xyz="0.064 -0.065 0.094" rpy="0 0 0"/>

File: urdf/aruco/turtlebot3_aruco_2.urdf.xacro (robot description, xacro)
@@ -75,5 +75,5 @@
         <mesh filename="package://turtlebot3_description/meshes/wheels/right_tire.stl" scale="0.001 0.001 0.001"/>
       </geometry>
-      <material name="dark"/>
+      <material name="dark" />
     </visual>
     <collision>
@@ -164,4 +164,73 @@
     </inertial>
   </link>
+<gazebo reference="ball">
+     <material>Marker/White</material>
+     <turnGravityOff>false</turnGravityOff>
+ </gazebo>
+  <link name="ball">
+    <visual>
+      <origin xyz="0 0 0" rpy="0 0 0"/>
+      <geometry>
+             <box size="0.15 0.15 1e-5"/>
+      </geometry>
+         <material name="m_Blue">
+    <color rgba="0.0 0.0 0.0 1.0"/>
+    <lighting>1</lighting>
+  </material>
+    </visual>
+    <collision>
+      <origin xyz="0.015 0 -0.0065" rpy="0 0 0"/>
+      <geometry>
+        <cylinder length="0.0315" radius="0.055"/>
+      </geometry>
+    </collision>
+    <inertial>
+      <mass value="0.114" />
+      <origin xyz="0 0 0" />
+      <inertia ixx="0.001" ixy="0.0" ixz="0.0"
+               iyy="0.001" iyz="0.0"
+               izz="0.001" />
+    </inertial>
+  </link>
+  <joint name="base_scan_ball" type="fixed">
+    <parent link="base_scan"/>
+    <child link="ball"/>
+    <origin xyz="-0.14 0.0 -0.03" rpy="0 1.57 0"/>
+    <axis xyz="0 0 1"/>
+  </joint>
+<gazebo reference="aruco">
+     <material>Marker/Marker2</material>
+     <turnGravityOff>false</turnGravityOff>
+ </gazebo>
+  <link name="aruco">
+    <visual>
+      <origin xyz="0 0 0" rpy="0 0 0"/>
+      <geometry>
+             <box size="0.12 0.12 1e-5"/>
+      </geometry>
+         <material name="m_Blue">
+    <color rgba="0.0 0.0 0.0 1.0"/>
+  </material>
+    </visual>
+    <collision>
+      <origin xyz="0.015 0 -0.0065" rpy="0 0 0"/>
+      <geometry>
+        <cylinder length="0.0315" radius="0.055"/>
+      </geometry>
+    </collision>
+    <inertial>
+      <mass value="0.114" />
+      <origin xyz="0 0 0" />
+      <inertia ixx="0.001" ixy="0.0" ixz="0.0"
+               iyy="0.001" iyz="0.0"
+               izz="0.001" />
+    </inertial>
+  </link>
+  <joint name="aruco_scan_ball" type="fixed">
+    <parent link="ball"/>
+    <child link="aruco"/>
+    <origin xyz="-0.0 0.0 -0.001" rpy="0 0 0"/>
+    <axis xyz="0 0 1"/>
+  </joint>
   <joint name="camera_joint" type="fixed">
     <origin xyz="0.064 -0.065 0.094" rpy="0 0 0"/>

File: urdf/optimal/turtlebot3_waffle_target.urdf.xacro (robot description, xacro)
@@ -1,5 +1,5 @@
 <?xml version="1.0" ?>
 <robot name="turtlebot3_waffle" xmlns:xacro="http://ros.org/wiki/xacro">
-  <xacro:include filename="$(find turtlebot3_description)/urdf/common_properties.xacro"/>
+  <xacro:include filename="$(find multi-agents-formulation)/urdf/common_properties.xacro"/>
   <xacro:include filename="$(find multi-agents-formulation)/urdf/optimal/turtlebot3_waffle_target.gazebo.xacro"/>
   <xacro:property name="r200_cam_rgb_px" value="0.005"/>
